File: kicad/chessmate.kicad_pcb (KiCad board)
At the start: 2 copper layers, 70 x 125.5 mm, 37 parts, among them J1 SPKR, Q1 2N2222, Q2 2N2222, Q3 2N2222, Q4 2N2222, Q5 2N2222, SW1 F6, SW10 ENTER, SW11 CLEAR, SW12 H8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

Commit message: kicad updates
Parts:
- removed J1: SPKR, Connector_PinHeader_2.54mm:PinHeader_1x02_P2.54mm_Horizontal
- added C1: 220uF, Capacitor_THT:CP_Radial_D6.3mm_P2.50mm, F.Cu at (85.0, 25.5)
- added D1: 1N4148, Diode_THT:D_DO-35_SOD27_P7.62mm_Horizontal, F.Cu at (116.0, 29.0)
- added J2: Power Jack, Connector_BarrelJack:BarrelJack_Horizontal, F.Cu at (70.5, 33.0)
- added LS1: Speaker, Buzzer_Beeper:Buzzer_12x9.5RM7.6, F.Cu at (99.5, 22.2)
- added REF**: MountingHole_3.2mm_M3, MountingHole:MountingHole_3.2mm_M3, F.Cu at (116.0, 140.5)
- added REF**: MountingHole_3.2mm_M3, MountingHole:MountingHole_3.2mm_M3, F.Cu at (54.5, 140.5)
- added REF**: MountingHole_3.2mm_M3, MountingHole:MountingHole_3.2mm_M3, F.Cu at (116.0, 23.0)
- added REF**: MountingHole_3.2mm_M3, MountingHole:MountingHole_3.2mm_M3, F.Cu at (54.0, 23.0)
- moved R18 22.8 mm to (111.0, 27.5), turned to 90 degrees
- moved R1 6.91 mm to (60.5, 27.0), turned to 90 degrees
Connections:
- Q5 pad 3: Net-(Q5-C) -> Net-(D1-A)
- R18 pad 1: Net-(J1-Pin_2) -> +5V
- R18 pad 2: Net-(Q5-C) -> Net-(D1-K)
- U2 pad J5_1: unconnected-(U2-5V-PadJ5_1) -> +5V
Routing:
- net +5V: track 0.00 -> 117.2 mm
- net +3V3: track 146.2 -> 35.9 mm, vias 1 -> 0
- net Net-(D1-A): track 0.00 -> 26.6 mm
- net Net-(D1-K): track 0.00 -> 19.3 mm
- net /DIG1_PIN: track 62.7 -> 79.9 mm
- net Net-(J1-Pin_2): track 17.1 -> 0.00 mm
- net GND: track 168.2 -> 182.2 mm
- net /SEGD_PIN: track 24.4 -> 10.6 mm
- net /DIG3: track 41.3 -> 52.9 mm
- net /SEGF_PIN: track 48.5 -> 38.2 mm
- net /SOUND_PIN: track 83.9 -> 93.8 mm, vias 2 -> 1
- net /DIG2_PIN: track 45.5 -> 37.5 mm
- net Net-(Q5-C): track 7.14 -> 0.00 mm
- net /ROW0_PIN: track 124.7 -> 119.3 mm
- net /SEGA_PIN: track 66.5 -> 71.4 mm
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- added copper zone on F.Cu, net +3V3
