File: kicad/chessmate.kicad_sch (KiCad schematic)
At the start: 40 parts, among them J2 Power Jack, Q1 2N2222, Q2 2N2222, Q3 2N2222, Q4 2N2222, Q5 2N2222, SW1 F6, SW10 ENTER, SW11 CLEAR, SW12 H8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

Commit message: replace 7-seg footprint with pin headers
Parts:
- removed U1: CC56-12SURKWA, Display_7Segment:CA56-12SURKWA, symbol Display_Character:CC56-12SURKWA
- added J1: 7SegBtm, Connector_PinHeader_2.54mm:PinHeader_1x06_P2.54mm_Vertical, symbol Connector:Conn_01x06_Socket
- added J3: 7SegTop, Connector_PinHeader_2.54mm:PinHeader_1x06_P2.54mm_Vertical, symbol Connector:Conn_01x06_Socket
Connections:
- net C: now reaches R7.2
- net C: now also J1.4 (Pin_4)
- net B: now reaches R6.2
- net B: now also J3.6 (Pin_6)
- net F: now reaches R10.2
- net F: now also J3.3 (Pin_3)
- net A: now reaches R5.2
- net A: now also J3.2 (Pin_2)
- net DP: now reaches R12.2
- net DP: now also J1.3 (Pin_3)
- net G: now reaches R11.2
- net G: now also J1.5 (Pin_5)
- net E: now reaches R9.2
- net E: now also J1.1 (Pin_1)
- net D: now reaches R8.2
- net D: now also J1.2 (Pin_2)
- net DIG1 renamed D1
- net D1: now also J3.1 (Pin_1)
- net DIG2 renamed D2
- net D2: now also J3.4 (Pin_4)
- net DIG3 renamed D3
- net D3: now also J3.5 (Pin_5)
- net DIG4 renamed D4
- net D4: now also J1.6 (Pin_6)
